File: Schematic/Nixie/Nixie.kicad_sch (KiCad schematic)
At the start: 0 parts

Commit message: schematics in progress
Parts:
- added A1: Arduino_Uno_R4_WiFi_Shield, PCM_arduino-library:Arduino_Uno_R4_WiFi_Shield, symbol PCM_arduino-library:Arduino_Uno_R4_WiFi_Shield
- added Nixie_IN-1, Nixie_IN-2, Nixie_IN-3, Nixie_IN-4, Nixie_IN-5, Nixie_IN-6: (no value), custom:Nixie_IN14, symbol custom:Nixie_IN14
- added R1, R2, R3, R4, R5, R6: 22k, symbol Device:R
- added R10, R11, R7, R8, R9: 10k, symbol PCM_Elektuur:R
- added SW1: RotaryEncoder_Switch, symbol Device:RotaryEncoder_Switch
- added SW2, SW3: SW_Push, Button_Switch_THT:SW_DIP_SPSTx01_Piano_10.8x4.1mm_W7.62mm_P2.54mm, symbol Switch:SW_Push
- added U1, U2: HV5122PG-G, QFP44_10x10MC_MCH, symbol custom:HV5122PG-G
- added U3: DS3231MZ, Package_SO:SOIC-8_3.9x4.9mm_P1.27mm, symbol Timer_RTC:DS3231MZ
- added U4: CD4504BE, N16, symbol custom:CD4504BE
- added U5: MOC3020M, symbol Relay_SolidState:MOC3020M
Connections:
- new net: Nixie_IN-1.1 (Anode), R1.2
- new net: Nixie_IN-2.1 (Anode), R2.2
- new net: Nixie_IN-4.1 (Anode), R4.2
- new net: Nixie_IN-6.1 (Anode), R6.2
- new net: Nixie_IN-3.1 (Anode), R3.2
- new net: Nixie_IN-5.1 (Anode), R5.2
- new net +12V: U1.31 (VDD), U2.31 (VDD), U4.16 (VDD)
- new net +180V: U5.6
- new net 3.3V: A1.3V3 (3.3V), R8.1 (+), R9.1 (+), SW1.S1
- new net 5V: A1.VIN, SW2.2, SW3.2, U3.2 (VCC), U3.6 (VBAT), U4.1 (VCC)
- new net CLK 12V: U1.29 (CLK), U2.29 (CLK), U4.2 (AOUT)
- new net CLK 5V: A1.A0, U4.3 (AIN)
- new net DATA 12V: U1.33 (DATAIN), U2.33 (DATAIN), U4.4 (BOUT)
- new net DATA 5V: A1.D8, U4.5 (BIN)
- new net GND: A1.GND1 (GND), A1.GND2 (GND), A1.GND3 (GND), A1.GND4 (GND), A1.GND5 (GND), R10.2 (-), R11.2 (-), R7.2 (-), SW1.C, U1.30 (GND), U2.30 (GND), U3.5 (GND), U5.2
- new net HVV-GND: R1.1, R2.1, R3.1, R4.1, R5.1, R6.1
- new net LE 12V: U1.32 (STR), U2.32 (STR), U4.6 (COUT)
- new net LE 5V: A1.D10, U4.7 (CIN)
- new net N1-03: Nixie_IN-1.3 (Cathode(1)), U1.1 (HVOUT11)
- new net N1-04: Nixie_IN-1.4 (Cathode(2)), U1.2 (HVOUT12)
- new net N1-05: Nixie_IN-1.5 (Cathode(3)), U1.3 (HVOUT13)
- new net N1-06: Nixie_IN-1.6 (Cathode(4)), U1.4 (HVOUT14)
- new net N1-07: Nixie_IN-1.7 (Cathode(5)), U1.5 (HVOUT15)
- new net N1-08: Nixie_IN-1.8 (Cathode(6)), U1.6 (HVOUT16)
- new net N1-09: Nixie_IN-1.9 (Cathode(7)), U1.7 (HVOUT17)
- new net N1-10: Nixie_IN-1.10 (Cathode(8)), U1.8 (HVOUT18)
- new net N1-11: Nixie_IN-1.11 (Cathode(9)), U1.9 (HVOUT19)
- new net N1-12: Nixie_IN-1.12 (Cathode(0)), U1.10 (HVOUT20)
- new net N2-03: Nixie_IN-2.3 (Cathode(1)), U1.11 (HVOUT21)
- new net N2-04: Nixie_IN-2.4 (Cathode(2)), U1.12 (HVOUT22)
- new net N2-05: Nixie_IN-2.5 (Cathode(3)), U1.13 (HVOUT23)
- new net N2-06: Nixie_IN-2.6 (Cathode(4)), U1.14 (HVOUT24)
- new net N2-07: Nixie_IN-2.7 (Cathode(5)), U1.15 (HVOUT25)
- new net N2-08: Nixie_IN-2.8 (Cathode(6)), U1.16 (HVOUT26)
- new net N2-09: Nixie_IN-2.9 (Cathode(7)), U1.17 (HVOUT27)
- new net N2-10: Nixie_IN-2.10 (Cathode(8)), U1.18 (HVOUT28)
- new net N2-11: Nixie_IN-2.11 (Cathode(9)), U1.19 (HVOUT29)
- new net N2-12: Nixie_IN-2.12 (Cathode(0)), U1.20 (HVOUT30)
- new net N3-03: Nixie_IN-3.3 (Cathode(1)), U1.44 (HVOUT10)
- new net N3-04: Nixie_IN-3.4 (Cathode(2)), U1.43 (HVOUT9)
- new net N3-05: Nixie_IN-3.5 (Cathode(3)), U1.42 (HVOUT8)
- new net N3-06: Nixie_IN-3.6 (Cathode(4)), U1.41 (HVOUT7)
- new net N3-07: Nixie_IN-3.7 (Cathode(5)), U1.40 (HVOUT6)
- new net N3-08: Nixie_IN-3.8 (Cathode(6)), U1.39 (HVOUT5)
- new net N3-09: Nixie_IN-3.9 (Cathode(7)), U1.38 (HVOUT4)
- new net N3-10: Nixie_IN-3.10 (Cathode(8)), U1.37 (HVOUT3)
- new net N3-11: Nixie_IN-3.11 (Cathode(9)), U1.36 (HVOUT2)
- new net N3-12: Nixie_IN-3.12 (Cathode(0)), U1.35 (HVOUT1)
- new net N4-03: Nixie_IN-4.3 (Cathode(1)), U2.1 (HVOUT11)
- new net N4-04: Nixie_IN-4.4 (Cathode(2)), U2.2 (HVOUT12)
- new net N4-05: Nixie_IN-4.5 (Cathode(3)), U2.3 (HVOUT13)
- new net N4-06: Nixie_IN-4.6 (Cathode(4)), U2.4 (HVOUT14)
- new net N4-07: Nixie_IN-4.7 (Cathode(5)), U2.5 (HVOUT15)
- new net N4-08: Nixie_IN-4.8 (Cathode(6)), U2.6 (HVOUT16)
- new net N4-09: Nixie_IN-4.9 (Cathode(7)), U2.7 (HVOUT17)
- new net N4-10: Nixie_IN-4.10 (Cathode(8)), U2.8 (HVOUT18)
- new net N4-11: Nixie_IN-4.11 (Cathode(9)), U2.9 (HVOUT19)
- new net N4-12: Nixie_IN-4.12 (Cathode(0)), U2.10 (HVOUT20)
- new net N5-03: Nixie_IN-5.3 (Cathode(1)), U2.11 (HVOUT21)
- new net N5-04: Nixie_IN-5.4 (Cathode(2)), U2.12 (HVOUT22)
- new net N5-05: Nixie_IN-5.5 (Cathode(3)), U2.13 (HVOUT23)
- new net N5-06: Nixie_IN-5.6 (Cathode(4)), U2.14 (HVOUT24)
- new net N5-07: Nixie_IN-5.7 (Cathode(5)), U2.15 (HVOUT25)
- new net N5-08: Nixie_IN-5.8 (Cathode(6)), U2.16 (HVOUT26)
- new net N5-09: Nixie_IN-5.9 (Cathode(7)), U2.17 (HVOUT27)
- new net N5-10: Nixie_IN-5.10 (Cathode(8)), U2.18 (HVOUT28)
- new net N5-11: Nixie_IN-5.11 (Cathode(9)), U2.19 (HVOUT29)
- new net N5-12: Nixie_IN-5.12 (Cathode(0)), U2.20 (HVOUT30)
- new net N6-03: Nixie_IN-6.3 (Cathode(1)), U2.44 (HVOUT10)
- new net N6-04: Nixie_IN-6.4 (Cathode(2)), U2.43 (HVOUT9)
- new net N6-05: Nixie_IN-6.5 (Cathode(3)), U2.42 (HVOUT8)
- new net N6-06: Nixie_IN-6.6 (Cathode(4)), U2.41 (HVOUT7)
- new net N6-07: Nixie_IN-6.7 (Cathode(5)), U2.40 (HVOUT6)
- new net N6-08: Nixie_IN-6.8 (Cathode(6)), U2.39 (HVOUT5)
- new net N6-09: Nixie_IN-6.9 (Cathode(7)), U2.38 (HVOUT4)
- new net N6-10: Nixie_IN-6.10 (Cathode(8)), U2.37 (HVOUT3)
- new net N6-11: Nixie_IN-6.11 (Cathode(9)), U2.36 (HVOUT2)
- new net N6-12: Nixie_IN-6.12 (Cathode(0)), U2.35 (HVOUT1)
- new net Nx-02: Nixie_IN-1.2 (Cathode(PL)), Nixie_IN-2.2 (Cathode(PL)), Nixie_IN-3.2 (Cathode(PL)), Nixie_IN-4.2 (Cathode(PL)), Nixie_IN-5.2 (Cathode(PL)), Nixie_IN-6.2 (Cathode(PL)), U1.21 (HVOUT31)
- new net Nx-13: Nixie_IN-1.13 (Cathode(PR)), Nixie_IN-2.13 (Cathode(PR)), Nixie_IN-3.13 (Cathode(PR)), Nixie_IN-4.13 (Cathode(PR)), Nixie_IN-5.13 (Cathode(PR)), Nixie_IN-6.13 (Cathode(PR)), U1.22 (HVOUT32)
- new net OE +180V: U1.28 (OE), U2.28 (OE), U5.4
- new net OE 5V: A1.D9, U5.1
- new net ROTARY A: A1.D11, R8.2 (-), SW1.A
- new net ROTARY B: A1.D12, R9.2 (-), SW1.B
- new net ROTARY SW: A1.D13, R7.1 (+), SW1.S2
- new net SCL: A1.SCL, U3.8 (SCL)
- new net SDA: A1.SDA, U3.7 (SDA)
- new net SW A: A1.D7, R10.1 (+), SW3.1
- new net SW B: A1.D6, R11.1 (+), SW2.1
- no-connect marks 0 -> 38
